File: hw/clockgen.sch (KiCad schematic (older format))
At the start: 14 parts

Commit message: more control signals
Connections:
- net labels added: -CTCLR
Changed lines of the file:
@@
 	1    0    0    -1
 $EndComp
-Text Notes 6400 6450 0    60   ~ 0
+Text Notes 6250 6550 0    60   ~ 0
 OLED display
 Text Label 4100 4550 0    60   ~ 0
@@
 	1    0    0    -1
 $EndComp
-Text Label 3450 3450 0    60   ~ 0
+Text Label 2600 3450 0    60   ~ 0
 -FASTEN
-Text Label 4400 5450 0    60   ~ 0
+Text Label 950  4350 0    60   ~ 0
 RST
-Text Label 4400 5550 0    60   ~ 0
+Text Label 950  4550 0    60   ~ 0
 -RST
 $Comp
@@
 Text Label 4350 5250 0    60   ~ 0
 -FASTEN
-Text Label 4400 5350 0    60   ~ 0
-SLOWCLK
 Wire Wire Line
 	4300 1550 5050 1550
@@
 	650  1600 900  1600
 Wire Wire Line
-	650  1000 650  1300
-Wire Wire Line
-	650  1300 650  1600
+	650  1000 650  1600
 Wire Wire Line
 	5850 6550 5250 6550
@@
 	4900 6450 4900 6550
 Wire Wire Line
-	2200 1300 2800 1300
-Wire Wire Line
-	2800 1300 3200 1300
+	2200 1300 3200 1300
 Wire Wire Line
 	3200 1050 2800 1050
@@
 	3200 1200 2900 1200
 Wire Wire Line
-	2900 950  2900 1200
-Wire Wire Line
-	2900 1200 2900 1500
+	2900 950  2900 1500
 Wire Wire Line
 	3200 950  2900 950
@@
 	5600 5150 5600 5400
 Wire Wire Line
-	5600 5400 5900 5400
-Wire Wire Line
-	5900 5400 6200 5400
-Wire Wire Line
-	6200 5400 6500 5400
-Wire Wire Line
-	6500 5400 6750 5400
-Wire Wire Line
-	6200 5150 6200 5400
-Wire Wire Line
-	6200 5400 6200 5550
+	5600 5400 6750 5400
+Wire Wire Line
+	6200 5150 6200 5550
 Wire Wire Line
 	6750 5400 6750 5150
@@
 	4050 5150 4450 5150
 Wire Bus Line
-	4550 2550 4550 2650
-Wire Bus Line
-	4550 2650 4550 2750
-Wire Bus Line
-	4550 2750 4550 4850
-Wire Bus Line
-	4550 4850 4550 4950
-Wire Bus Line
-	4550 4950 4550 5050
+	4550 2550 4550 5050
 Wire Wire Line
 	5050 2450 4650 2450
@@
 	6900 1900 6900 3450
 Wire Wire Line
-	6900 3450 4900 3450
-Wire Wire Line
-	4900 3450 3400 3450
+	6900 3450 2550 3450
 Wire Wire Line
 	5050 2850 4900 2850
@@
 Connection ~ 4900 3450
 Wire Wire Line
-	4800 5450 4050 5450
-Wire Wire Line
-	4800 5550 4050 5550
+	1350 4350 600  4350
+Wire Wire Line
+	1350 4550 600  4550
 Wire Wire Line
 	7750 4700 7200 4700
@@
 	7750 4900 7200 4900
 Wire Wire Line
-	8950 4800 9050 4800
-Wire Wire Line
-	9050 4800 11050 4800
+	8950 4800 11050 4800
 Wire Wire Line
 	9350 5100 9050 5100
@@
 Wire Wire Line
 	5150 4550 5150 6650
+Wire Wire Line
+	4050 5450 4800 5450
+Text Label 4350 5350 0    60   ~ 0
+-CTCLR
+Wire Wire Line
+	3200 1400 3200 3300
+Wire Wire Line
+	2550 3300 7900 3300
+Text Label 2600 3300 0    60   ~ 0
+-CTCLR
+Wire Wire Line
+	8400 2700 7900 2700
+Wire Wire Line
+	7900 2700 7900 3300
+Connection ~ 3200 3300
+Text Label 4400 5450 0    60   ~ 0
+SLOWCLK
+Wire Wire Line
+	8400 2000 8250 2000
+Wire Wire Line
+	8250 2000 8250 2850
+$Comp
+L GND #PWR?
+U 1 1 599C87C9
+P 8250 2850
+F 0 "#PWR?" H 8250 2600 50  0001 C CNN
+F 1 "GND" H 8250 2700 50  0000 C CNN
+F 2 "" H 8250 2850 50  0000 C CNN
+F 3 "" H 8250 2850 50  0000 C CNN
+	1    8250 2850
+	1    0    0    -1
+$EndComp
+Wire Wire Line
+	8400 2200 8250 2200
+Connection ~ 8250 2200
+Wire Wire Line
+	8400 2400 8250 2400
+Connection ~ 8250 2400
 $EndSCHEMATC

Commit message: use atmega328 with Arduino runtime support
This is most likely the easiest way to use the
OLED display.
Parts:
- removed IC?: ATTINY2313A-P, DIP20, symbol ATTINY2313A-P
- added C? (x2): C, symbol C
- added D?: LED, symbol LED
- added R? (x2): R, symbol R
- added SW?: SW_PUSH, symbol SW_PUSH
- added U?: ATMEGA328-PU, DIL28, symbol ATMEGA328-PU
- added Y?: Crystal, symbol Crystal
Connections:
- net labels added: AVRRST, RX, TX, XTAL1, XTAL2
- wire segments 82 -> 125
Other:
- note added: "Crystal osc"
- note added: "Reset button"
- moved on the sheet: P?, SW?, U?, U?A, U?C, U?D

Commit message: basic circuit is in place?
Parts:
- added R? (x2): R, symbol R
- added U?: 74LS02, symbol 74LS02
Connections:
- wire segments 125 -> 114
Other:
- note added: "RX/TX go to FT232\nboard (USB serial)"
- note added: "flexible clock generator"
- note added: "unused gate"
- moved on the sheet: C?, D?, P?, R?, SW?, U?, Y?

Commit message: specify component designators
Parts:
- removed D?: LED, symbol LED
- added D1: LED, symbol LED
- C1, C2: renamed from C?; value C -> 22pF
- R2, R3, R4: renamed from R?; value R -> 4K7
- U2: renamed from U?; value 74LS590 -> 74HC590
- U3: renamed from U?; value 74LS151 -> 74HC151
- U4: renamed from U?; value 74LS02 -> 74HC02
- U5: renamed from U?; value 74LS175 -> 74HC175
- gave numbers to parts that had none: 10
Other:
- moved on the sheet: R1
Changed lines of the file:
@@
 $EndDescr
 $Comp
-L 74LS590 U?
+L 74LS590 U2
 U 1 1 599C3081
 P 4750 2050
-F 0 "U?" H 5050 2850 50  0000 C CNN
-F 1 "74LS590" H 5000 1300 50  0000 C CNN
+F 0 "U2" H 5050 2850 50  0000 C CNN
+F 1 "74HC590" H 5000 1300 50  0000 C CNN
 F 2 "" H 4750 2050 60  0000 C CNN
 F 3 "" H 4750 2050 60  0000 C CNN
@@
 $EndComp
 $Comp
-L 74LS151 U?
+L 74LS151 U3
 U 1 1 599C30EA
 P 6750 2650
-F 0 "U?" H 6750 2650 50  0000 C CNN
-F 1 "74LS151" H 6750 2500 50  0000 C CNN
+F 0 "U3" H 6750 2650 50  0000 C CNN
+F 1 "74HC151" H 6750 2500 50  0000 C CNN
 F 2 "" H 6750 2650 50  0000 C CNN
 F 3 "" H 6750 2650 50  0000 C CNN
@@
 $EndComp
 $Comp
-L XTAL_OSC_HALF_CAN U?
+L XTAL_OSC_HALF_CAN U1
 U 1 1 599C32CC
 P 2800 1900
-F 0 "U?" H 2800 2200 60  0000 C CNN
+F 0 "U1" H 2800 2200 60  0000 C CNN
 F 1 "XTAL_OSC_HALF_CAN" H 2800 1600 60  0000 C CNN
 F 2 "" H 2800 1900 60  0000 C CNN
@@
 $EndComp
 $Comp
-L SW_PUSH SW?
+L SW_PUSH SW1
 U 1 1 599C413A
 P 4250 5650
-F 0 "SW?" H 4400 5760 50  0000 C CNN
+F 0 "SW1" H 4400 5760 50  0000 C CNN
 F 1 "SW_PUSH" H 4250 5570 50  0000 C CNN
 F 2 "" H 4250 5650 50  0000 C CNN
@@
 $EndComp
 $Comp
-L SW_PUSH SW?
+L SW_PUSH SW2
 U 1 1 599C41F1
 P 4550 5650
-F 0 "SW?" H 4700 5760 50  0000 C CNN
+F 0 "SW2" H 4700 5760 50  0000 C CNN
 F 1 "SW_PUSH" H 4550 5570 50  0000 C CNN
 F 2 "" H 4550 5650 50  0000 C CNN
@@
 $EndComp
 $Comp
-L SW_PUSH SW?
+L SW_PUSH SW3
 U 1 1 599C426D
 P 4850 5650
-F 0 "SW?" H 5000 5760 50  0000 C CNN
+F 0 "SW3" H 5000 5760 50  0000 C CNN
 F 1 "SW_PUSH" H 4850 5570 50  0000 C CNN
 F 2 "" H 4850 5650 50  0000 C CNN
@@
 $EndComp
 $Comp
-L SW_PUSH SW?
+L SW_PUSH SW4
 U 1 1 599C4273
 P 5150 5650
-F 0 "SW?" H 5300 5760 50  0000 C CNN
+F 0 "SW4" H 5300 5760 50  0000 C CNN
 F 1 "SW_PUSH" H 5150 5570 50  0000 C CNN
 F 2 "" H 5150 5650 50  0000 C CNN
@@
 $EndComp
 $Comp
-L SW_PUSH SW?
+L SW_PUSH SW5
 U 1 1 599C465A
 P 5400 5650
-F 0 "SW?" H 5550 5760 50  0000 C CNN
+F 0 "SW5" H 5550 5760 50  0000 C CNN
 F 1 "SW_PUSH" H 5400 5570 50  0000 C CNN
 F 2 "" H 5400 5650 50  0000 C CNN
@@
 $EndComp
 $Comp
-L 74LS175 U?
+L 74LS175 U5
 U 1 1 599C4EB5
 P 9800 2700
-F 0 "U?" H 9800 2700 50  0000 C CNN
-F 1 "74LS175" H 9900 2300 50  0000 C CNN
+F 0 "U5" H 9800 2700 50  0000 C CNN
+F 1 "74HC175" H 9900 2300 50  0000 C CNN
 F 2 "" H 9800 2700 50  0000 C CNN
 F 3 "" H 9800 2700 50  0000 C CNN
@@
 FASTCLK
 $Comp
-L 74LS02 U?
+L 74LS02 U4
 U 1 1 599C5A4B
 P 8350 2250
-F 0 "U?" H 8350 2300 50  0000 C CNN
-F 1 "74LS02" H 8400 2200 50  0000 C CNN
+F 0 "U4" H 8350 2300 50  0000 C CNN
+F 1 "74HC02" H 8400 2200 50  0000 C CNN
 F 2 "" H 8350 2250 50  0000 C CNN
 F 3 "" H 8350 2250 50  0000 C CNN
@@
 -RST
 $Comp
-L 74LS02 U?
+L 74LS02 U4
 U 4 1 599C659F
 P 8750 1000
-F 0 "U?" H 8750 1050 50  0000 C CNN
-F 1 "74LS02" H 8800 950 50  0000 C CNN
+F 0 "U4" H 8750 1050 50  0000 C CNN
+F 1 "74HC02" H 8800 950 50  0000 C CNN
 F 2 "" H 8750 1000 50  0000 C CNN
 F 3 "" H 8750 1000 50  0000 C CNN
@@
 $EndComp
 $Comp
-L 74LS02 U?
+L 74LS02 U4
 U 3 1 599C66D6
 P 10050 1400
-F 0 "U?" H 10050 1450 50  0000 C CNN
-F 1 "74LS02" H 10100 1350 50  0000 C CNN
+F 0 "U4" H 10050 1450 50  0000 C CNN
+F 1 "74HC02" H 10100 1350 50  0000 C CNN
 F 2 "" H 10050 1400 50  0000 C CNN
 F 3 "" H 10050 1400 50  0000 C CNN
@@
 TX
 $Comp
-L LED D?
-U 1 1 599D23F7
-P 3150 4400
-F 0 "D?" H 3150 4500 50  0000 C CNN
-F 1 "LED" H 3150 4300 50  0000 C CNN
-F 2 "" H 3150 4400 50  0001 C CNN
-F 3 "" H 3150 4400 50  0001 C CNN
-	1    3150 4400
-	0    -1   -1   0
-$EndComp
-$Comp
-L R R?
+L R R1
 U 1 1 599D24C7
-P 3150 4000
-F 0 "R?" V 3230 4000 50  0000 C CNN
-F 1 "R" V 3150 4000 50  0000 C CNN
-F 2 "" V 3080 4000 50  0001 C CNN
-F 3 "" H 3150 4000 50  0001 C CNN
-	1    3150 4000
-	1    0    0    -1
-$EndComp
-Wire Wire Line
-	3150 4250 3150 4150
+P 3150 3900
+F 0 "R1" V 3230 3900 50  0000 C CNN
+F 1 "R" V 3150 3900 50  0000 C CNN
+F 2 "" V 3080 3900 50  0001 C CNN
+F 3 "" H 3150 3900 50  0001 C CNN
+	1    3150 3900
+	1    0    0    -1
+$EndComp
+Wire Wire Line
+	3150 4150 3150 4050
 Wire Wire Line
 	3150 4550 3150 5350
 Wire Wire Line
-	3150 3850 3150 3750
+	3150 3750 3150 3650
 $Comp
 L VCC #PWR?
 U 1 1 599D26C5
-P 3150 3750
-F 0 "#PWR?" H 3150 3600 50  0001 C CNN
-F 1 "VCC" H 3150 3900 50  0000 C CNN
-F 2 "" H 3150 3750 50  0001 C CNN
-F 3 "" H 3150 3750 50  0001 C CNN
-	1    3150 3750
+P 3150 3650
+F 0 "#PWR?" H 3150 3500 50  0001 C CNN
+F 1 "VCC" H 3150 3800 50  0000 C CNN
+F 2 "" H 3150 3650 50  0001 C CNN
+F 3 "" H 3150 3650 50  0001 C CNN
+	1    3150 3650
 	1    0    0    -1
 $EndComp
@@
 	9450 5250 9450 5200
 $Comp
-L R R?
+L R R4
 U 1 1 599D0902
 P 9450 5050
-F 0 "R?" V 9530 5050 50  0000 C CNN
-F 1 "R" V 9450 5050 50  0000 C CNN
+F 0 "R4" V 9530 5050 50  0000 C CNN
+F 1 "4K7" V 9450 5050 50  0000 C CNN
 F 2 "" V 9380 5050 50  0001 C CNN
 F 3 "" H 9450 5050 50  0001 C CNN
@@
 	8900 5250 9450 5250
 $Comp
-L SW_PUSH SW?
+L SW_PUSH SW6
 U 1 1 599D0583
 P 9450 5550
-F 0 "SW?" H 9600 5660 50  0000 C CNN
+F 0 "SW6" H 9600 5660 50  0000 C CNN
 F 1 "SW_PUSH" H 9450 5470 50  0000 C CNN
 F 2 "" H 9450 5550 50  0000 C CNN
@@
 $EndComp
 $Comp
-L C C?
+L C C2
 U 1 1 599CCB90
 P 7150 5550
-F 0 "C?" H 7175 5650 50  0000 L CNN
-F 1 "C" H 7175 5450 50  0000 L CNN
+F 0 "C2" H 7175 5650 50  0000 L CNN
+F 1 "22pF" H 7175 5450 50  0000 L CNN
 F 2 "" H 7188 5400 50  0001 C CNN
 F 3 "" H 7150 5550 50  0001 C CNN
@@
 $EndComp
 $Comp
-L C C?
+L C C1
 U 1 1 599CCAB2
 P 7150 5250
-F 0 "C?" H 7175 5350 50  0000 L CNN
-F 1 "C" H 7175 5150 50  0000 L CNN
+F 0 "C1" H 7175 5350 50  0000 L CNN
+F 1 "22pF" H 7175 5150 50  0000 L CNN
 F 2 "" H 7188 5100 50  0001 C CNN
 F 3 "" H 7150 5250 50  0001 C CNN
@@
 $EndComp
 $Comp
-L Crystal Y?
+L Crystal Y1
 U 1 1 599CC479
 P 6750 5400
-F 0 "Y?" H 6750 5550 50  0000 C CNN
+F 0 "Y1" H 6750 5550 50  0000 C CNN
 F 1 "Crystal" H 6750 5250 50  0000 C CNN
 F 2 "" H 6750 5400 50  0001 C CNN
@@
 SCL
 $Comp
-L ATMEGA328-PU U?
+L ATMEGA328-PU U6
 U 1 1 599CC266
 P 1900 5950
-F 0 "U?" H 1150 7200 50  0000 L BNN
+F 0 "U6" H 1150 7200 50  0000 L BNN
 F 1 "ATMEGA328-PU" H 2300 4550 50  0000 L BNN
 F 2 "DIL28" H 1900 5950 50  0001 C CIN
@@
 flexible clock generator
 $Comp
-L R R?
+L R R2
 U 1 1 599D04B4
 P 3700 5850
-F 0 "R?" V 3780 5850 50  0000 C CNN
-F 1 "R" V 3700 5850 50  0000 C CNN
+F 0 "R2" V 3780 5850 50  0000 C CNN
+F 1 "4K7" V 3700 5850 50  0000 C CNN
 F 2 "" V 3630 5850 50  0001 C CNN
 F 3 "" H 3700 5850 50  0001 C CNN
@@
 $EndComp
 $Comp
-L R R?
+L R R3
 U 1 1 599D0605
 P 3900 5850
-F 0 "R?" V 3980 5850 50  0000 C CNN
-F 1 "R" V 3900 5850 50  0000 C CNN
+F 0 "R3" V 3980 5850 50  0000 C CNN
+F 1 "4K7" V 3900 5850 50  0000 C CNN
 F 2 "" V 3830 5850 50  0001 C CNN
 F 3 "" H 3900 5850 50  0001 C CNN
@@
 $EndComp
 $Comp
-L 74LS02 U?
+L 74LS02 U4
 U 2 1 599D0A9C
 P 10550 5300
-F 0 "U?" H 10550 5350 50  0000 C CNN
-F 1 "74LS02" H 10600 5250 50  0000 C CNN
+F 0 "U4" H 10550 5350 50  0000 C CNN
+F 1 "74HC02" H 10600 5250 50  0000 C CNN
 F 2 "" H 10550 5300 50  0001 C CNN
 F 3 "" H 10550 5300 50  0001 C CNN
@@
 Text Notes 10150 4950 0    60   ~ 0
 unused gate
+$Comp
+L LED D1
+U 1 1 59A9A757
+P 3150 4350
+F 0 "D1" H 3150 4450 50  0000 C CNN
+F 1 "LED" H 3150 4250 50  0000 C CNN
+F 2 "" H 3150 4350 50  0000 C CNN
+F 3 "" H 3150 4350 50  0000 C CNN
+	1    3150 4350
+	0    -1   -1   0
+$EndComp
 $EndSCHEMATC

Commit message: use 74HC74 as the flip flop
Parts:
- removed U5: 74HC175, symbol 74LS175
- added U5: 74HC74, symbol 74LS74
- added U?: 74LS74, symbol 74LS74
- D1: symbol LED -> LED-RESCUE-clockgen
Connections:
- wire segments 114 -> 118
Other:
- note added: "unused gates"
- note removed: "unused gate"
- moved on the sheet: C1, C2, P?, R4, SW6, U4B, U4C, U4D, Y1
